File: reflow_V7.kicad_sch (KiCad schematic)
At the start: 60 parts

Commit message: update PCB
Parts:
- added C11, C15: 100nF, Capacitor_SMD:C_0805_2012Metric_Pad1.18x1.45mm_HandSolder, symbol Device:C_Small
- added C12, C16: 10uF/10V, Capacitor_Tantalum_SMD:CP_EIA-3216-10_Kemet-I_Pad1.58x1.35mm_HandSolder, symbol Device:C_Polarized_Small
- added C17, C18: 100uF, Capacitor_SMD:C_0805_2012Metric_Pad1.18x1.45mm_HandSolder, symbol Device:C
- added D10, D9: LED, LED_SMD:LED_0805_2012Metric_Pad1.15x1.40mm_HandSolder, symbol Device:LED
- added D7, D8: SS24, Diode_SMD:D_SMA, symbol Diode:B120-E3
- added J4, J5: THERMAL, Connector_PinHeader_2.54mm:PinHeader_1x02_P2.54mm_Vertical, symbol Connector_Generic:Conn_01x02
- added J6: Conn_01x03, Connector_PinHeader_2.54mm:PinHeader_1x03_P2.54mm_Vertical, symbol Connector_Generic:Conn_01x03
- added R20, R27: 4K7, Resistor_SMD:R_0805_2012Metric_Pad1.20x1.40mm_HandSolder, symbol Device:R_Small
- added R24, R28: 22R, Resistor_SMD:R_0805_2012Metric_Pad1.20x1.40mm_HandSolder, symbol Device:R_Small
- added R29: 1K, Resistor_SMD:R_0805_2012Metric_Pad1.20x1.40mm_HandSolder, symbol Device:R_Small_US
- added R30: 220, Resistor_SMD:R_0805_2012Metric_Pad1.20x1.40mm_HandSolder, symbol Device:R_Small_US
- added U3: AMS1117-3.3, Package_TO_SOT_SMD:SOT-223-3_TabPin2, symbol Regulator_Linear:AMS1117-3.3
- D1: renamed from D?; footprint (none) -> LED_SMD:LED_0805_2012Metric_Pad1.15x1.40mm_HandSolder
- D3, D5: renamed from D?; footprint Diode_SMD:D_SMA_Handsoldering -> Diode_SMD:D_SMA
- FAN1: renamed from FAN; footprint (none) -> TerminalBlock:TerminalBlock_bornier-2_P5.08mm
- Q1, Q2, Q3, Q4: renamed from Q?; footprint (none) -> Package_TO_SOT_SMD:SOT-23
- R11, R12: renamed from R?; value 10K -> 4K7
- SSR1, SSR2: footprint (none) -> TerminalBlock:TerminalBlock_bornier-2_P5.08mm
- gave numbers to parts that had none: 47
- renumbered RESET to RESET1
Connections:
- net +12V: now also J3.2 (Pin_2), D7.1 (K), R29.1; no longer J3.1 (Pin_1)
- net +3V3: now also C18.1, R20.1, R27.1, R30.1, U3.2 (VO)
- net +5V: now also J3.1 (Pin_1), C17.1, D8.1 (K), U3.3 (VI); no longer J3.2 (Pin_2)
- net ADC1: now also R24.1
- net ADC2: now also R28.1
- net BUZZER: now also R14.1, R16.1
- net FAN: no longer R14.1, R16.1
- net GND: now also C11.2, C12.2, C15.2, C16.2, C17.2, C18.2, D10.1 (K), D9.1 (K), J4.1 (Pin_1), J5.1 (Pin_1), J6.1 (Pin_1), U3.1 (GND)
- new net: D9.2 (A), R29.2
- new net: C11.1, C12.1, J4.2 (Pin_2), R20.2, R24.2
- new net: C15.1, C16.1, J5.2 (Pin_2), R27.2, R28.2
- new net: D7.2 (A), J6.3 (Pin_3)
- new net: D10.2 (A), R30.2
- new net: D8.2 (A), J6.2 (Pin_2)
Other:
- moved on the sheet: C13, C14, D1, R25, R26, R5, SW3, SW4
